Commit message: ns, controller added. not working

File: tfm_gazebo/urdf/quadrotor.urdf.xacro (robot description, xacro)
@@ -1,3 +1,3 @@
-<?xml version="1.0"?>
+﻿<?xml version="1.0"?>
 <robot name="quadrotor"
     xmlns:sensor="http://playerstage.sourceforge.net/gazebo/xmlschema/#sensor"
@@ -5,6 +5,6 @@
 xmlns:xacro="http://ros.org/wiki/xacro">
     <!-- Included URDF Files -->
-    <xacro:include filename="$(find cvg_sim_gazebo)/urdf/quadrotor_base.urdf.xacro" />
+    <xacro:include filename="$(find tfm_gazebo)/urdf/quadrotor_base.urdf.xacro" />
     <!-- Instantiate quadrotor_base_macro once (has no parameters atm) -->
-    <quadrotor_base_macro />
+    <quadrotor_base_macro ns="${ns}"/>
 </robot>

File: tfm_gazebo/urdf/quadrotor_base.urdf.xacro (robot description, xacro)
@@ -1,3 +1,3 @@
-<?xml version="1.0"?>
+﻿<?xml version="1.0"?>
 <robot xmlns:sensor="http://playerstage.sourceforge.net/gazebo/xmlschema/#sensor"
 xmlns:controller="http://playerstage.sourceforge.net/gazebo/xmlschema/#controller"
@@ -5,5 +5,5 @@
   <xacro:include filename="$(find cvg_sim_gazebo_plugins)/urdf/quadrotor_plugins.urdf.xacro" />
   <!-- Main quadrotor link -->
-  <xacro:macro name="quadrotor_base_macro">
+  <xacro:macro name="quadrotor_base_macro" params="ns">
     <link name="base_link">
       <inertial>
@@ -15,5 +15,5 @@
         <origin xyz="0 0 0" rpy="0 0 0" />
         <geometry>
-          <mesh filename="package://cvg_sim_gazebo/meshes/quadrotor/quadrotor_4.dae"/>
+          <mesh filename="package://tfm_gazebo/meshes/quadrotor/quadrotor_4.dae"/>
         </geometry>
       </visual>
@@ -21,5 +21,5 @@
         <origin xyz="0 0 0" rpy="0 0 0" />
         <geometry>
-          <mesh filename="package://cvg_sim_gazebo/meshes/quadrotor/quadrotor_4.stl"/>
+          <mesh filename="package://tfm_gazebo/meshes/quadrotor/quadrotor_4.stl"/>
         </geometry>
       </collision>
@@ -29,5 +29,5 @@
     </gazebo>
     <!-- Gazebo Plugins -->
-    <quadrotor_plugins/>
+    <quadrotor_plugins ns="${ns}"/>
   </xacro:macro>
 </robot>

File: tfm_gazebo/urdf/quadrotor_sensors.urdf.xacro (robot description, xacro)
@@ -1,3 +1,3 @@
-<?xml version="1.0"?>
+﻿<?xml version="1.0"?>
 <robot name="quadrotor_hokuyo_utm30lx"
 xmlns:sensor="http://playerstage.sourceforge.net/gazebo/xmlschema/#sensor"
@@ -6,14 +6,14 @@
     <xacro:property name="M_PI" value="3.1415926535897931" />
     <!-- Included URDF Files -->
-    <xacro:include filename="$(find cvg_sim_gazebo)/urdf/quadrotor_base.urdf.xacro" />
+    <xacro:include filename="$(find tfm_gazebo)/urdf/quadrotor_base.urdf.xacro" />
     <!-- Instantiate quadrotor_base_macro once (has no parameters atm) -->
-    <quadrotor_base_macro />
+    <quadrotor_base_macro ns="$(arg ns)"/>
     <!-- Sonar height sensor -->
-    <xacro:include filename="$(find cvg_sim_gazebo)/urdf/sensors/sonar_sensor.urdf.xacro" />
+    <xacro:include filename="$(find tfm_gazebo)/urdf/sensors/sonar_sensor.urdf.xacro" />
     <xacro:sonar_sensor name="sonar" parent="base_link" ros_topic="sonar_height" update_rate="10" min_range="0.01" max_range="3.0" field_of_view="${40*M_PI/180}" ray_count="3">
       <origin xyz="-0.15 0.0 0.0" rpy="0 ${90*M_PI/180} 0"/>
     </xacro:sonar_sensor>
     <!-- Hokuyo UTM-30LX mounted upside down below the quadrotor body
-    <xacro:include filename="$(find cvg_sim_gazebo)/urdf/sensors/hokuyo_utm30lx.urdf.xacro" />
+    <xacro:include filename="$(find tfm_gazebo)/urdf/sensors/hokuyo_utm30lx.urdf.xacro" />
     <xacro:hokuyo_utm30lx name="laser0" parent="base_link" ros_topic="scan" update_rate="40" ray_count="1081" min_angle="135" max_angle="-135">
       <origin xyz="0.0 0.0 0.08" rpy="${M_PI} 0 0"/>
@@ -21,11 +21,11 @@
     <!-- The following two cameras should be united to one! -->
     <!-- Forward facing camera -->
-    <xacro:include filename="$(find cvg_sim_gazebo)/urdf/sensors/generic_camera.urdf.xacro" />
-    <xacro:generic_camera name="front" sim_name="ardrone" parent="base_link" update_rate="60" res_x="640" res_y="360" image_format="R8G8B8" hfov="${81*M_PI/180}">
+    <xacro:include filename="$(find tfm_gazebo)/urdf/sensors/generic_camera.urdf.xacro" />
+    <xacro:generic_camera name="front" sim_name="$(arg ns)" parent="base_link" update_rate="60" res_x="640" res_y="360" image_format="R8G8B8" hfov="${81*M_PI/180}">
       <origin xyz="0.21 0.0 0.01" rpy="0 0 0"/>
     </xacro:generic_camera>
     <!-- Downward facing camera -->
-    <xacro:include filename="$(find cvg_sim_gazebo)/urdf/sensors/generic_camera.urdf.xacro" />
-    <xacro:generic_camera name="bottom" sim_name="ardrone" parent="base_link" update_rate="60" res_x="640" res_y="360" image_format="R8G8B8" hfov="${81*M_PI/180}">
+    <xacro:include filename="$(find tfm_gazebo)/urdf/sensors/generic_camera.urdf.xacro" />
+    <xacro:generic_camera name="bottom" sim_name="$(arg ns)" parent="base_link" update_rate="60" res_x="640" res_y="360" image_format="R8G8B8" hfov="${81*M_PI/180}">
         <origin xyz="0.15 0.0 0.0" rpy="0 ${M_PI/2} 0"/>
     </xacro:generic_camera>

File: tfm_gazebo/urdf/sensors/hokuyo_utm30lx.urdf.xacro (robot description, xacro)
@@ -18,5 +18,5 @@
 	  <origin xyz="0 0 0" rpy="0 0 0" />
           <geometry>
-          <mesh filename="package://cvg_sim_gazebo/meshes/hokuyo_utm30lx/hokuyo_utm_30lx$(optenv TEST_SELF_FILTER).dae"/>
+          <mesh filename="package://tfm_gazebo/meshes/hokuyo_utm30lx/hokuyo_utm_30lx$(optenv TEST_SELF_FILTER).dae"/>
         </geometry>
 	</visual>

File: tfm_gazebo/urdf/sensors/sonar_sensor.urdf.xacro (robot description, xacro)
@@ -19,5 +19,5 @@
         <geometry>
           <!--<box size="0.01 0.01 0.01" /> -->
-          <mesh filename="package://cvg_sim_gazebo/meshes/sonar_sensor/max_sonar_ez4.dae"/>
+          <mesh filename="package://tfm_gazebo/meshes/sonar_sensor/max_sonar_ez4.dae"/>
         </geometry>
       </visual>
